File: p-rot3-mx/PCB/Lily58_prot_MX.kicad_pcb (KiCad board)
At the start: 2 copper layers, 142.5 x 106.3 mm, 84 parts, among them J1 LED, J2 4PIN, J3 OLED, P1 i2c_pin, P2 i2c_pin, SW1 SW_PUSH, SW10 SW_PUSH, SW11 SW_PUSH, SW12 SW_PUSH, SW13 SW_PUSH, SW14 SW_PUSH, SW15 SW_PUSH, SW16 SW_PUSH, SW17 SW_PUSH, SW18 SW_PUSH, SW19 SW_PUSH, SW2 SW_PUSH, SW20 SW_PUSH, SW21 SW_PUSH, SW22 SW_PUSH, SW23 SW_PUSH, SW24 SW_PUSH, SW25 SW_PUSH, SW26 SW_PUSH, SW27 SW_PUSH, SW28 SW_PUSH, SW29 SW_PUSH, SW3 SW_PUSH, SW30 ROT_ENC_SW, SW4 SW_PUSH, SW5 SW_PUSH, SW6 SW_PUSH, SW7 SW_PUSH, SW8 SW_PUSH, SW9 SW_PUSH, U1 ProMicro

Commit message: added extra encoders to schematic and PCB -- still need to be routed; diodes now SOD
Parts:
- added SW31: ROT_ENC_SW, Lily58_prot_MX-footprint:RotaryEncoder_Alps_EC11E-Switch_Vertical_H20mm-keebio_modified-no_MP, F.Cu at (168.1, 123.8)
- added SW32: ROT_ENC_SW, Lily58_prot_MX-footprint:RotaryEncoder_Alps_EC11E-Switch_Vertical_H20mm-keebio_modified-no_MP, F.Cu at (215.7, 53.9)
- D1, D10, D11, D12, D13, D14, D15, D16, D17, D18, D19, D2, D20, D21, D22, D23, D24, D25, D26, D27, D28, D29, D3, D4, D5, D6, D7, D8, D9: footprint Lily58_prot_MX-footprint:Diode_TH_SOD123 -> Lily58_prot_MX-footprint:Diode_SOD123
- moved D29 19.2 mm to (162.8, 114.3)
- moved D27 17.9 mm to (136.3, 117.2)
- moved D28 17.8 mm to (152.9, 115.4)
- moved D13 11.9 mm to (128.9, 90.3), turned to 90 degrees
- moved D25 11.7 mm to (109.3, 100.3), turned to 90 degrees
- moved D5 11.6 mm to (204.9, 54.7), turned to 90 degrees
- moved D17 11.5 mm to (205.1, 92.6), turned to 90 degrees
- moved D19 11.3 mm to (128.9, 109.3), turned to 90 degrees
- moved D18 11.3 mm to (207.4, 94.0), turned to 90 degrees
- moved D1 11.1 mm to (128.9, 52.5), turned to 90 degrees
- moved D16 11.0 mm to (186.1, 87.9), turned to 90 degrees
- moved D21 10.9 mm to (167.0, 105.6), turned to 90 degrees
- moved D22 10.9 mm to (185.9, 107.0), turned to 90 degrees
- moved D8 10.9 mm to (147.8, 68.9), turned to 90 degrees
- moved D9 10.9 mm to (166.9, 67.6), turned to 90 degrees
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Connections:
- net Net-(D29-Pad2) renamed R2_SW1
- net Net-(D6-Pad2) renamed R3_SW1
- net R_SW1 renamed R1_SW1
- net R_SW2 renamed R1_SW2
- net col0 renamed R3_SW2
- net col1 renamed R2_SW2
Routing:
- net R_A: track 81.8 -> 289.6 mm
- net R_B: track 89.0 -> 182.8 mm
- net GND: track 152.3 -> 103.1 mm
- net row2: track 166.3 -> 144.0 mm
- net row3: track 184.0 -> 162.7 mm, vias 2 -> 1
- net R1_SW1: track 35.1 -> 18.0 mm
- net row4: track 143.5 -> 127.9 mm, vias 2 -> 1
- net row1: track 140.5 -> 125.4 mm
- net Net-(D17-Pad2): track 23.5 -> 10.3 mm
- net Net-(D13-Pad2): track 23.6 -> 10.4 mm
- net Net-(D19-Pad2): track 23.2 -> 10.2 mm
- net Net-(D16-Pad2): track 23.5 -> 10.5 mm
- net Net-(D5-Pad2): track 23.6 -> 10.7 mm
- net Net-(D14-Pad2): track 23.2 -> 10.5 mm
- net Net-(D21-Pad2): track 22.8 -> 10.2 mm
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
Commit message: added routing for GND to all encoders
Parts:
- moved D6 16.5 mm to (224.0, 56.1)
- moved D12 0.46 mm to (207.5, 75.0)
Connections:
- SW32 pad A: R_A -> R_B
- SW32 pad B: R_B -> R_A
Routing:
- net GND: track 103.1 -> 357.1 mm
- net R_B: track 182.8 -> 292.1 mm, vias 0 -> 1
- net row0: track 123.8 -> 140.0 mm
- net R3_SW1: track 32.7 -> 16.6 mm
- net LED: track 57.0 -> 71.0 mm
- net R_A: track 289.6 -> 291.0 mm, vias 2 -> 3
- net col2: track 250.4 -> 249.2 mm

Commit message: rerouted all switch, encoder, and ground traces
Parts:
- moved D29 20.3 mm to (175.9, 129.7), turned to 90 degrees
- moved D24 16.3 mm to (223.5, 113.5)
- moved D18 16.1 mm to (223.5, 94.4)
- moved D12 16.0 mm to (223.5, 75.6)
- moved D28 15.7 mm to (157.5, 130.4), turned to 90 degrees
- moved D25 15.7 mm to (94.0, 103.3)
- moved D26 13.9 mm to (107.1, 135.5), turned to 30 degrees
- moved D27 11.7 mm to (138.4, 128.7), turned to 90 degrees
- moved D6 2.62 mm to (223.5, 58.6)
- moved D5 0.80 mm to (205.1, 55.5)
- moved D2 0.41 mm to (148.0, 51.0)
- moved D1 0.41 mm to (128.9, 52.9)
- moved D3 0.41 mm to (167.0, 49.7)
Connections:
- SW32 pad A: R_B -> R_A
- SW32 pad B: R_A -> R_B
Routing:
- net GND: track 357.1 -> 402.8 mm, vias 4 -> 28
- net row4: track 127.9 -> 166.1 mm
- net R_A: track 291.0 -> 270.4 mm, vias 3 -> 2
- net Net-(D24-Pad2): track 28.9 -> 10.9 mm
- net Net-(D18-Pad2): track 28.7 -> 11.0 mm
- net Net-(D12-Pad2): track 28.1 -> 11.0 mm
- net row1: track 125.3 -> 141.9 mm
- net R1_SW1: track 18.0 -> 33.9 mm
- net LED: track 71.0 -> 55.1 mm
- net col3: track 236.8 -> 222.9 mm
- net col2: track 249.2 -> 239.1 mm
- net row2: track 144.0 -> 152.8 mm
- net R_B: track 292.1 -> 283.9 mm
- net R2_SW1: track 26.4 -> 18.5 mm
- net row3: track 162.7 -> 170.5 mm
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