File: prot3mx/PCB/Lily58_prot_MX.kicad_pcb (KiCad board)
At the start: 2 copper layers, 142.5 x 106.3 mm, 87 parts, among them J1 LED, J2 4PIN, J3 OLED, P1 i2c_pin, P2 i2c_pin, SW1 SW_PUSH, SW10 SW_PUSH, SW11 SW_PUSH, SW12 SW_PUSH, SW13 SW_PUSH, SW14 SW_PUSH, SW15 SW_PUSH, SW16 SW_PUSH, SW17 SW_PUSH, SW18 SW_PUSH, SW19 SW_PUSH, SW2 SW_PUSH, SW20 SW_PUSH, SW21 SW_PUSH, SW22 SW_PUSH, SW23 SW_PUSH, SW24 SW_PUSH, SW25 SW_PUSH, SW26 SW_PUSH, SW27 SW_PUSH, SW28 SW_PUSH, SW29 SW_PUSH, SW3 SW_PUSH, SW30 ROT_ENC_SW, SW31 ROT_ENC_SW, SW32 ROT_ENC_SW, SW4 SW_PUSH, SW5 SW_PUSH, SW6 SW_PUSH, SW7 SW_PUSH, SW8 SW_PUSH, SW9 SW_PUSH, U1 ProMicro

Commit message: minor rerouting for greater ground plane coverage; also moved bottow row diodes to be centred with upper row diodes.
Parts:
- moved D25 8.26 mm to (153.5, 116.6)
- moved D26 8.26 mm to (156.1, 116.7)
- moved D27 8.26 mm to (158.5, 116.7)
- moved D28 8.26 mm to (160.9, 116.7)
- moved D29 8.26 mm to (163.3, 116.7)
Routing:
- net row4: track 110.8 -> 120.5 mm
- net R1_SW1: track 72.3 -> 81.6 mm
- net Net-(D27-Pad2): track 41.6 -> 49.8 mm
- net Net-(D26-Pad2): track 57.8 -> 66.0 mm
- net R_A: track 351.2 -> 359.0 mm
- net Net-(D28-Pad2): track 24.6 -> 31.5 mm
- net R2_SW1: track 24.7 -> 19.8 mm
- net GND: track 75.4 -> 77.5 mm, vias 31 -> 44
- net col2: track 260.1 -> 258.2 mm
- net R_B: track 347.4 -> 348.3 mm
- net Net-(D9-Pad2): track 17.7 -> 18.4 mm

Commit message: added modified Lily58 silkscreen logo to board; generated gerber files as per JLC instructions.
Parts:
- added G***: LOGO, Lily58_prot_MX-footprint:lily58Pro.3RE.MX-logo, F.Cu at (96.9, 81.7)
Routing:
- net row0: track 91.0 -> 95.7 mm
- net Net-(D8-Pad2): track 35.8 -> 36.6 mm
- net Net-(D1-Pad2): track 54.0 -> 53.4 mm
- net Net-(D9-Pad2): track 18.4 -> 18.9 mm
- net GND: vias 44 -> 46
Other:
- rule pad_to_mask_clearance: 0.2 -> 0
- board text added: "JLCJLCJLCJLC"
